File: esp32_octal_wled.kicad_sch (KiCad schematic)
At the start: 70 parts, among them J1 LED1, J11 I2C EXT, J12 ATX-24, J13 LED1, J14 LED1, J15 LED1, J16 LED1, J17 BH1750 (0x23), J18 BME280 (0x76), J2 LED1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

Commit message: OctalWLED as ordered @ JLCPCB
Connections:
- net +3V3: now also J11.2 (Pin_2); no longer J11.1 (Pin_1)
- net GND: now also J11.1 (Pin_1); no longer J11.2 (Pin_2)
Changed lines of the file:
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@@
 	(symbol
 		(lib_id "power:GND")
-		(at 83.82 86.36 270)
+		(at 83.82 83.82 270)
 		(unit 1)
 		(exclude_from_sim no)
@@
 		(dnp no)
 		(property "Reference" "#PWR039"
-			(at 77.47 86.36 0)
+			(at 77.47 83.82 0)
 			(effects
 				(font
@@
 		)
 		(property "Value" "GND"
-			(at 79.4258 86.487 90)
+			(at 79.4258 83.947 90)
 			(effects
 				(font
@@
 		)
 		(property "Footprint" ""
-			(at 83.82 86.36 0)
+			(at 83.82 83.82 0)
 			(effects
 				(font
@@
 		)
 		(property "Datasheet" ""
-			(at 83.82 86.36 0)
+			(at 83.82 83.82 0)
 			(effects
 				(font
@@
 		)
 		(property "Description" ""
-			(at 83.82 86.36 0)
+			(at 83.82 83.82 0)
 			(effects
 				(font
@@
 	(symbol
 		(lib_id "power:+3V3")
-		(at 83.82 83.82 90)
+		(at 83.82 86.36 90)
 		(unit 1)
 		(exclude_from_sim no)
@@
 		(dnp no)
 		(property "Reference" "#PWR040"
-			(at 87.63 83.82 0)
+			(at 87.63 86.36 0)
 			(effects
 				(font
@@
 		)
 		(property "Value" "+3V3"
-			(at 78.74 83.82 90)
+			(at 78.74 86.36 90)
 			(effects
 				(font
@@
 		)
 		(property "Footprint" ""
-			(at 83.82 83.82 0)
+			(at 83.82 86.36 0)
 			(effects
 				(font
@@
 		)
 		(property "Datasheet" ""
-			(at 83.82 83.82 0)
+			(at 83.82 86.36 0)
 			(effects
 				(font
@@
 		)
 		(property "Description" ""
-			(at 83.82 83.82 0)
-			(effects
-				(font
+			(at 83.82 86.36 0)
+			(effects
+				(font

Commit message: Minor fixes
Parts:
- J13: value LED1 -> LED5
- J14: value LED1 -> LED6
- J15: value LED1 -> LED7
- J16: value LED1 -> LED8
- J2: value LED1 -> LED2
- J6: value LED1 -> LED3
- J7: value LED1 -> LED4
Changed lines of the file:
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@@
 			)
 		)
-		(property "Value" "LED1"
+		(property "Value" "LED4"
 			(at 274.32 49.5299 0)
 			(effects
@@
 			)
 		)
-		(property "Value" "LED1"
+		(property "Value" "LED8"
 			(at 274.32 85.0899 0)
 			(effects
@@
 			)
 		)
-		(property "Value" "LED1"
+		(property "Value" "LED3"
 			(at 274.32 40.6399 0)
 			(effects
@@
 			)
 		)
-		(property "Value" "LED1"
+		(property "Value" "LED7"
 			(at 274.32 76.1999 0)
 			(effects
@@
 			)
 		)
-		(property "Value" "LED1"
+		(property "Value" "LED6"
 			(at 274.32 67.3099 0)
 			(effects
@@
 			)
 		)
-		(property "Value" "LED1"
+		(property "Value" "LED2"
 			(at 274.32 31.7499 0)
 			(effects
@@
 			)
 		)
-		(property "Value" "LED1"
+		(property "Value" "LED5"
 			(at 274.32 58.4199 0)
 			(effects

Commit message: WIP
Parts:
- added JP1: -, Jumper:SolderJumper-2_P1.3mm_Bridged2Bar_Pad1.0x1.5mm, symbol Jumper:Jumper_2_Bridged
- added Q1: AO3400A, Package_TO_SOT_SMD:SOT-23_Handsoldering, symbol Transistor_FET:AO3400A
- added R13: 10k, Resistor_SMD:R_0805_2012Metric_Pad1.20x1.40mm_HandSolder, symbol Device:R
- added R15: k1, Resistor_SMD:R_0805_2012Metric_Pad1.20x1.40mm_HandSolder, symbol Device:R
- J3: footprint Connector:Tag-Connect_TC2030-IDC-NL_2x03_P1.27mm_Vertical -> liebler_CONN:IDC_2x03_P1.27mm_Vertical
Connections:
- net GND: now also JP1.1 (A), Q1.2 (S), R13.1; no longer J1.3 (Pin_3)
- net STRIP1: now also U2.11 (DAC_2/ADC2_CH9/GPIO26); no longer U2.12 (ADC2_CH7/GPIO27)
- net STRIP4: now also U2.12 (ADC2_CH7/GPIO27); no longer U2.11 (DAC_2/ADC2_CH9/GPIO26)
- net STRIP_5V_1: now also R15.2
- new net: Q1.1 (G), R13.2, R15.1
- new net STRIP_GND_1: J1.3 (Pin_3), JP1.2 (B), Q1.3 (D)
Other:
- note added: "v2) Strip 1 und 4 getauscht!"

Commit message: New Version as ordered @ JLCPCB
Parts:
- added Q3, Q4: IRLZ44N, Package_TO_SOT_THT:TO-220-3_Vertical, symbol Transistor_FET:IRLZ44N
- added R16, R18: k1, Resistor_SMD:R_0805_2012Metric_Pad1.20x1.40mm_HandSolder, symbol Device:R
- added R17, R19: 10k, Resistor_SMD:R_0805_2012Metric_Pad1.20x1.40mm_HandSolder, symbol Device:R
- C1: value m1 -> 10u; footprint Capacitor_SMD:C_1206_3216Metric_Pad1.33x1.80mm_HandSolder -> Capacitor_SMD:C_0805_2012Metric_Pad1.18x1.45mm_HandSolder; JLCPCB C15008 -> (none)
- C2: value 10u -> u1
- C5: now left out of the parts list
- JP1: value - -> STRIP1
- R2: value 22k -> 15k
- R3: value 15k -> 10k
Connections:
- net 485_DI: now also U2.9 (32K_XN/GPIO33/ADC1_CH5); no longer U2.10 (DAC_1/ADC2_CH8/GPIO25)
- net GND: now also J4.2 (Pin_2), Q3.3 (S), Q4.3 (S), R17.1, R19.1; no longer J4.1 (Pin_1), J6.3 (Pin_3), J7.3 (Pin_3)
- net I2S_SCK: now also U2.10 (DAC_1/ADC2_CH8/GPIO25); no longer U2.9 (32K_XN/GPIO33/ADC1_CH5)
- net RS485A: now also J4.3 (Pin_3), R1.1; no longer J4.2 (Pin_2), SW1.1 (A)
- net RS485B: now also J4.1 (Pin_1), SW1.2 (B), SW1.3 (C); no longer J4.3 (Pin_3), R1.1
- net STRIP_5V_3: now also R16.2
- net STRIP_5V_4: now also R18.2
- net at R1.2: now also SW1.1 (A); no longer SW1.2 (B)
- new net: Q4.1 (G), R18.1, R19.2
- new net: Q3.1 (G), R16.1, R17.2
- new net STRIP_GND_3: J6.3 (Pin_3), Q3.2 (D)
- new net STRIP_GND_4: J7.3 (Pin_3), Q4.2 (D)
Other:
- moved on the sheet: H1, H2, H3, H4, R1
