File: esp32_octal_wled.kicad_pcb (KiCad board)
At the start: 2 copper layers, 90 x 48.9 mm, 70 parts, among them J1 LED1, J11 I2C EXT, J12 ATX-24, J13 LED1, J14 LED1, J15 LED1, J16 LED1, J17 BH1750 (0x23), J18 BME280 (0x76), J2 LED1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

Commit message: Minor fixes
Parts:
- J13: value LED1 -> LED5
- J14: value LED1 -> LED6
- J15: value LED1 -> LED7
- J16: value LED1 -> LED8
- J2: value LED1 -> LED2
- J6: value LED1 -> LED3
- J7: value LED1 -> LED4

Commit message: WIP
Parts:
- added JP1: -, Jumper:SolderJumper-2_P1.3mm_Bridged2Bar_Pad1.0x1.5mm, F.Cu at (110.6, 137.3)
- added Q1: AO3400A, Package_TO_SOT_SMD:SOT-23_Handsoldering, F.Cu at (114.2, 138.6)
- added R13: 10k, Resistor_SMD:R_0805_2012Metric_Pad1.20x1.40mm_HandSolder, F.Cu at (117.9, 138.6)
- added R15: k1, Resistor_SMD:R_0805_2012Metric_Pad1.20x1.40mm_HandSolder, F.Cu at (105.2, 140.4)
- J3: footprint Connector:Tag-Connect_TC2030-IDC-NL_2x03_P1.27mm_Vertical -> liebler_CONN:IDC_2x03_P1.27mm_Vertical
- moved R7 28.1 mm to (160.5, 108.5)
- moved C10 18.3 mm to (128.0, 127.8), turned to -90 degrees
- moved U3 14.6 mm to (124.4, 121.8), turned to -90 degrees
- moved J17 13.0 mm to (169.1, 110.6), turned to 90 degrees
- moved J18 11.2 mm to (157.1, 115.6), turned to 180 degrees
- moved U9 10.7 mm to (115.0, 114.2), turned to 0 degrees
- moved R2 8.97 mm to (165.9, 126.5), turned to 180 degrees
- moved R14 8.64 mm to (117.0, 118.3), turned to 0 degrees
- moved R3 8.27 mm to (162.2, 126.5), turned to 180 degrees
- moved R6 7.70 mm to (174.5, 108.7), turned to 90 degrees
- moved R5 6.40 mm to (172.6, 108.7), turned to 90 degrees
- moved Q2 4.81 mm to (131.8, 125.7)
- moved C11 4.70 mm to (172.5, 121.8), turned to -90 degrees
- moved C13 4.41 mm to (159.3, 122.8)
- moved J3 3.86 mm to (162.7, 114.2), turned to -90 degrees
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Connections:
- J1 pad 3: GND -> /STRIP_GND_1
- U2 pad 11: STRIP4 -> STRIP1
- U2 pad 12: STRIP1 -> STRIP4
Routing:
- net +5V: track 126.7 -> 40.6 mm, vias 1 -> 0
- net GND: track 167.2 -> 98.1 mm, vias 153 -> 110
- net Onewire: track 24.5 -> 42.9 mm
- net STRIP2: track 30.2 -> 13.0 mm
- net STRIP3: track 33.2 -> 16.6 mm
- net STRIP1: track 23.9 -> 10.4 mm
- net Net-(Q1-G): track 0.00 -> 12.9 mm
- net STRIP4: track 27.3 -> 14.8 mm
- net STRIP_5V_4: track 11.5 -> 21.9 mm
- net STRIP_5V_7: track 30.4 -> 20.8 mm
- net Net-(J12-PWR_OK): track 17.2 -> 9.52 mm
- net STRIP5: track 27.0 -> 20.0 mm
- net STRIP6: track 31.8 -> 25.0 mm
- net STRIP_5V_5: track 9.26 -> 15.8 mm
- net STRIP_5V_6: track 6.03 -> 11.1 mm
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
Commit message: New Version as ordered @ JLCPCB
Parts:
- removed C5: m1, Capacitor_SMD:C_1206_3216Metric_Pad1.33x1.80mm_HandSolder
- added Q3: IRLZ44N, Package_TO_SOT_THT:TO-220-3_Vertical, B.Cu at (116.1, 117.6)
- added Q4: IRLZ44N, Package_TO_SOT_THT:TO-220-3_Vertical, B.Cu at (121.0, 117.6)
- added R16: k1, Resistor_SMD:R_0805_2012Metric_Pad1.20x1.40mm_HandSolder, F.Cu at (114.2, 118.5)
- added R17: 10k, Resistor_SMD:R_0805_2012Metric_Pad1.20x1.40mm_HandSolder, F.Cu at (112.3, 117.3)
- added R18: k1, Resistor_SMD:R_0805_2012Metric_Pad1.20x1.40mm_HandSolder, F.Cu at (118.8, 116.9)
- added R19: 10k, Resistor_SMD:R_0805_2012Metric_Pad1.20x1.40mm_HandSolder, F.Cu at (123.9, 117.7)
- C1: value m1 -> 10u; footprint Capacitor_SMD:C_1206_3216Metric_Pad1.33x1.80mm_HandSolder -> Capacitor_SMD:C_0805_2012Metric_Pad1.18x1.45mm_HandSolder
- C2: value 10u -> u1
- JP1: value - -> STRIP1
- R2: value 22k -> 15k
- R3: value 15k -> 10k
- moved R1 21.8 mm to (124.6, 111.3), turned to 180 degrees
- moved U9 20.6 mm to (132.8, 124.6), turned to -90 degrees
- moved R4 19.2 mm to (140.5, 139.7)
- moved R11 17.9 mm to (156.7, 126.5), turned to 0 degrees
- moved C3 17.7 mm to (156.1, 138.4), turned to 90 degrees
- moved C9 17.3 mm to (179.9, 147.7)
- moved F8 15.9 mm to (186.9, 141.0), turned to -90 degrees
- moved F1 15.9 mm to (103.1, 143.8), turned to 90 degrees
- moved C4 15.8 mm to (154.1, 138.4), turned to 90 degrees
- moved R15 14.7 mm to (119.8, 138.6), turned to 90 degrees
- moved R14 13.7 mm to (128.7, 125.6), turned to 180 degrees
- moved Q2 13.6 mm to (135.9, 138.7), turned to 180 degrees
- moved R12 12.8 mm to (176.1, 147.7), turned to 0 degrees
- moved U10 9.20 mm to (105.2, 110.5)
- moved C1 9.10 mm to (167.9, 137.9), turned to 0 degrees
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Connections:
- J4 pad 1: GND -> RS485B
- J4 pad 2: RS485A -> GND
- J4 pad 3: RS485B -> RS485A
- J6 pad 3: GND -> /STRIP_GND_3
- J7 pad 3: GND -> /STRIP_GND_4
- R1 pad 1: RS485B -> RS485A
- R1 pad 2: Net-(SW1-B) -> Net-(SW1-A)
- SW1 pad 1: RS485A -> Net-(SW1-A)
- SW1 pad 2: Net-(SW1-B) -> RS485B
- SW1 pad 3: unconnected-(SW1-C-Pad3) -> RS485B
- U2 pad 10: 485_DI -> I2S_SCK
- U2 pad 9: I2S_SCK -> 485_DI
Routing:
- net +12V: track 69.1 -> 187.2 mm
- net +5V: track 40.6 -> 91.5 mm
- net Onewire: track 42.9 -> 11.4 mm
- net +3V3: track 139.6 -> 169.9 mm, vias 28 -> 29
- net Net-(SW1-B): track 20.1 -> 0.00 mm
- net /STRIP_GND_4: track 0.00 -> 19.3 mm
- net PROG_IO0: track 51.8 -> 64.7 mm
- net GND: track 98.1 -> 85.5 mm, vias 110 -> 141
- net STRIP_5V_4: track 21.9 -> 31.7 mm, vias 0 -> 1
- net I2S_WS: track 4.31 -> 14.1 mm, vias 0 -> 1
- net I2S_SCK: track 4.31 -> 13.4 mm, vias 0 -> 1
- net STRIP_5V_1: track 44.7 -> 53.6 mm
- net Net-(Q1-G): track 12.9 -> 4.05 mm
- net Net-(SW1-A): track 0.00 -> 8.56 mm
- net /STRIP_GND_3: track 0.00 -> 8.39 mm
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Other:
- board text added: "Octal WLED Module Klaus Liebler 2026-01-09 MIT License"
- board text added: "SIG"
- board text added: "STRIP1 GND"
- board text added: "STRIP3 GND"
- board text removed: "MOVE"
- board text removed: "Octal WLED Module Klaus Liebler 2025-01-14 MIT License"
